Commit message: urdf change for cross platform compatibility

File: src/assets/urdf/satellite/urdf/satellite.urdf (robot description, URDF)
Before this commit: robot satellite, 4 links, 3 joints
Links:
- link base_link: geometry collision mesh filename=../meshes/base_link.STL; visual mesh filename=../meshes/base_link.STL
- link left_Link: geometry collision mesh filename=../meshes/left_Link.STL; visual mesh filename=../meshes/left_Link.STL
- link right_Link: geometry collision mesh filename=../meshes/right_Link.STL; visual mesh filename=../meshes/right_Link.STL

File: src/assets/urdf/satellite_battery/urdf/satellite_battery.urdf (robot description, URDF)
Before this commit: robot satellite_battery, 1 links, 0 joints
Links:
- link base_link: geometry collision mesh filename=../meshes/base_link.STL; visual mesh filename=../meshes/base_link.STL
